File: KICAD/Untitled/Untitled.kicad_sch (KiCad schematic)
At the start: 10 parts, among them J1 USB4105-GF-A, U1 ESP32-C3-MINI-1-N4, U2 DWM3000SQ

Commit message: v3
Parts:
- removed VR1: LM3940IMP-3.3/NOPB, VREG_LM3940IMP-3.3/NOPB, symbol LM3940IMP-3.3_NOPB:LM3940IMP-3.3/NOPB
- added D1, D2, D3, D4: LED, LED_SMD:LED_0603_1608Metric, symbol Device:LED
- added FID1, FID2, FID3, FID4: Fiducial, Fiducial:Fiducial_1mm_Mask2mm, symbol Mechanical:Fiducial
- added H1, H2, H3, H4: MountingHole, MountingHole:MountingHole_3.2mm_M3_DIN965_Pad, symbol Mechanical:MountingHole
- added JP2: SolderJumper_2_Open, Jumper:SolderJumper-2_P1.3mm_Open_Pad1.0x1.5mm, symbol Jumper:SolderJumper_2_Open
- added R10, R7, R8, R9: 1K, Resistor_SMD:R_0603_1608Metric, symbol Device:R
- added R11, R12, R13: 49.9R, Resistor_SMD:R_0603_1608Metric, symbol Device:R
- added R14, R6: 100K, Resistor_SMD:R_0603_1608Metric, symbol Device:R
- added R4, R5: 5k1, Resistor_SMD:R_0603_1608Metric, symbol Device:R
- added U4: AMS1117-3.3, Package_TO_SOT_SMD:SOT-223-3_TabPin2, symbol Regulator_Linear:AMS1117-3.3
- C1: footprint (none) -> Capacitor_SMD:C_0603_1608Metric; Order (none) -> https://www.mouser.com/ProductDetail/KEMET/C0603C105K4RACTU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
- C2: value 0.1u -> 10u; footprint (none) -> Capacitor_SMD:C_0603_1608Metric; Order (none) -> https://www.mouser.com/ProductDetail/Samsung-Electro-Mechan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
- C3: value 10u -> 22u; footprint (none) -> Capacitor_SMD:C_0603_1608Metric; Order (none) -> https://www.mouser.com/ProductDetail/Murata-Electronics/GRM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
- J1: Order (none) -> https://www.mouser.com/ProductDetail/GCT/USB4105-GF-A?qs=KU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
- R1: value 10K -> 49.9R; footprint (none) -> Resistor_SMD:R_0603_1608Metric; Order (none) -> https://www.mouser.com/ProductDetail/YAGEO/AF0603FR-0749R9L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
- R2, R3: footprint (none) -> Resistor_SMD:R_0603_1608Metric; Order (none) -> https://www.mouser.com/ProductDetail/Vishay-Draloric/RCG060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
- U1: Order https://www.mouser.com/ProductDetail/Espressif-Systems/ESP32-C3-MINI-1-N4?qs=stqOd1AaK7%252B/pH3qqyGehA%3D%3D -> https://www.mouser.com/ProductDetail/Espressif-Systems/ESP32-C3-MINI-1-N4?qs=sGAEpiMZZMu3sxpa5v1qrhrB%252BBlYHY1OkYOS7ceUJhQ%3D
- U2: Order (none) -> https://store.qorvo.com/products/detail/dwm3000-qorvo/68194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
Connections:
- net GND: now also J1.A1_B12 (GND), J1.B1_A12 (GND), U1.6 (IO3), U2.16 (VSS), U2.2 (WAKEUP), U2.21 (VSS), U2.23 (VSS), U2.24 (VSS), U2.8 (VSS), D1.1 (K), D2.1 (K), D3.1 (K), D4.1 (K), JP2.2 (B), R14.1, R4.2, R5.1, R6.2, U4.1 (GND)
- net SPICS: now reaches R1.2
- net SPICS: now also U1.16 (IO10); no longer U1.5 (IO2)
- net VBUS: now reaches J1.A4_B9 (VBUS), J1.B4_A9 (VBUS)
- net VBUS: now also C2.1, U4.3 (VI)
- net at J1.A5 (CC1): now also R5.2
- net D+: now reaches J1.A6 (DP1)
- net D+: now also J1.B6 (DP2), U1.27 (IO19)
- net D-: now reaches J1.A7 (DN1)
- net D-: now also J1.B7 (DN2), U1.26 (IO18)
- net at J1.B5 (CC2): now also R4.1
- net at J1.S1 (SHELL_GND), J1.S2 (SHELL_GND), J1.S3 (SHELL_GND)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: now also R6.1
- net RST_UWB: now reaches U1.18 (IO4)
- net RST_UWB: now also U2.3 (~{RST})
- net SPICLK: now reaches U1.20 (IO6)
- net SPICLK: now also R11.2
- net SPIMOSI: now reaches U1.21 (IO7)
- net SPIMOSI: now also R13.2
- net at U1.23 (IO9): now also JP2.1 (A)
- net at U2.12 (GPIO3/TXLED): now also R10.2
- net at U2.13 (GPIO2/RXLED): now also R7.2
- net at U2.14 (GPIO1/SFDLED): now also R8.2
- net at U2.15 (GPIO0/RXOKLED): now also R9.2
- net at U2.17 (~{SPICS}): now also R1.1
- net at U2.18 (SPIMOSI): now also R13.1
- net at U2.19 (SPIMISO): now also R12.1
- net at U2.20 (SPICLK): now also R11.1
- net at U2.22 (GPIO8/IRQ): now also R14.2
- net VDD: now reaches U2.5 (VDD1)
- net VDD: now also C1.1, C3.1, R2.1, R3.2, U1.3 (3V3), U2.6 (VDD3V3), U2.7 (VDD3V3), U4.2 (VO)
- removed net VDD33: C1.1, C2.1, C3.1, R1.1, R2.1, R3.2, U1.3 (3V3)
- new net: D1.2 (A), R10.1
- new net: D4.2 (A), R9.1
- new net: D3.2 (A), R8.1
- new net: D2.2 (A), R7.1
- new net SPIMISO: R12.2, U1.5 (IO2)
- no-connect marks 2 -> 12
Other:
- note added: "BONUS"
- note added: "MICROCONTROLLER"
- note added: "SENSOR"
- company: (none) -> Ben Stirling
- title: (none) -> AirPark
